Commit message: “增加f2的bvh重定向”

File: assets/f2/F1_1.urdf (robot description, URDF)
Before this commit: robot F2, 36 links, 34 joints
Links:
- removed link waist_roll_link
- link head_pitch_link: geometry visual mesh filename=meshes/head_pitch_link.STL
- link left_ankle_pitch_link: geometry collision mesh filename=meshes/left_ankle_pitch_link.STL; visual mesh filename=meshes/left_ankle_pitch_link.STL
- link left_ankle_roll_link: geometry collision mesh filename=meshes/left_ankle_roll_link.STL; visual mesh filename=meshes/left_ankle_roll_link.STL
- link left_elbow_link: geometry collision mesh filename=meshes/left_elbow_link.STL; visual mesh filename=meshes/left_elbow_link.STL
- link left_hand_link: geometry collision mesh filename=meshes/left_hand_link.STL; visual mesh filename=meshes/left_hand_link.STL
- link left_hip_pitch_link: geometry collision mesh filename=meshes/left_hip_pitch_link.STL; visual mesh filename=meshes/left_hip_pitch_link.STL
- link left_hip_roll_link: geometry collision mesh filename=meshes/left_hip_roll_link.STL; visual mesh filename=meshes/left_hip_roll_link.STL
- link left_hip_yaw_link: geometry collision mesh filename=meshes/left_hip_yaw_link.STL; visual mesh filename=meshes/left_hip_yaw_link.STL
- link left_knee_link: geometry collision mesh filename=meshes/left_knee_link.STL; visual mesh filename=meshes/left_knee_link.STL
- link left_shoulder_pitch_link: geometry collision mesh filename=meshes/left_shoulder_pitch_link.STL; visual mesh filename=meshes/left_shoulder_pitch_link.STL
- link left_shoulder_roll_link: geometry collision mesh filename=meshes/left_shoulder_roll_link.STL; visual mesh filename=meshes/left_shoulder_roll_link.STL
- link left_shoulder_yaw_link: geometry collision mesh filename=meshes/left_shoulder_yaw_link.STL; visual mesh filename=meshes/left_shoulder_yaw_link.STL
- link left_wrist_pitch_link: mass 0.042 -> 0.12; geometry visual mesh filename=meshes/left_wrist_pitch_link_v1_1.STL
- link left_wrist_roll_link: geometry collision mesh filename=meshes/left_wrist_roll_link_v1_1.STL; visual mesh filename=meshes/left_wrist_roll_link_v1_1.STL
- link left_wrist_yaw_link: mass 0.12 -> 0.042; geometry collision mesh filename=meshes/left_wrist_yaw_link_v1_1.STL; visual mesh filename=meshes/left_wrist_yaw_link_v1_1.STL
- link right_ankle_pitch_link: geometry collision mesh filename=meshes/right_ankle_pitch_link.STL; visual mesh filename=meshes/right_ankle_pitch_link.STL
- link right_ankle_roll_link: geometry collision mesh filename=meshes/right_ankle_roll_link.STL; visual mesh filename=meshes/right_ankle_roll_link.STL
- link right_elbow_link: geometry collision mesh filename=meshes/right_elbow_link.STL; visual mesh filename=meshes/right_elbow_link.STL
- link right_hand_link: geometry collision mesh filename=meshes/right_hand_link.STL; visual mesh filename=meshes/right_hand_link.STL
- link right_hip_pitch_link: geometry collision mesh filename=meshes/right_hip_pitch_link.STL; visual mesh filename=meshes/right_hip_pitch_link.STL
- link right_hip_roll_link: geometry collision mesh filename=meshes/right_hip_roll_link.STL; visual mesh filename=meshes/right_hip_roll_link.STL
- link right_hip_yaw_link: geometry collision mesh filename=meshes/right_hip_yaw_link.STL; visual mesh filename=meshes/right_hip_yaw_link.STL
- link right_knee_link: geometry collision mesh filename=meshes/right_knee_link.STL; visual mesh filename=meshes/right_knee_link.STL
- link right_shoulder_pitch_link: geometry collision mesh filename=meshes/right_shoulder_pitch_link.STL; visual mesh filename=meshes/right_shoulder_pitch_link.STL
- link right_shoulder_roll_link: geometry collision mesh filename=meshes/right_shoulder_roll_link.STL; visual mesh filename=meshes/right_shoulder_roll_link.STL
- link right_shoulder_yaw_link: geometry collision mesh filename=meshes/right_shoulder_yaw_link.STL; visual mesh filename=meshes/right_shoulder_yaw_link.STL
- link right_wrist_pitch_link: mass 0.042 -> 0.12; geometry visual mesh filename=meshes/right_wrist_pitch_link_v1_1.STL
- link right_wrist_roll_link: geometry collision mesh filename=meshes/right_wrist_roll_link_v1_1.STL; visual mesh filename=meshes/right_wrist_roll_link_v1_1.STL
- link right_wrist_yaw_link: mass 0.12 -> 0.042; geometry collision mesh filename=meshes/right_wrist_yaw_link_v1_1.STL; visual mesh filename=meshes/right_wrist_yaw_link_v1_1.STL
- link torso_link: geometry collision mesh filename=meshes/torso_link.STL; visual mesh filename=meshes/torso_link.STL
Joints:
- joint left_hand_joint: origin xyz=0.031 0 0 rpy=0 0 0 -> xyz=0.016 0 0 rpy=0 0 0; parent left_wrist_yaw_link -> left_wrist_pitch_link
- joint left_wrist_pitch_joint: limit lower=-0.5236 upper=0.5236 effort=20 velocity=6.28 -> lower=-0.5236 upper=0.5236 effort=25 velocity=4.44; origin xyz=0.23 0 0 rpy=0 0 0 -> xyz=0.021 0 0 rpy=0 0 0; parent left_wrist_roll_link -> left_wrist_yaw_link
- joint left_wrist_roll_joint: limit lower=-2.0071 upper=2.0071 effort=37 velocity=7.33 -> lower=-3.7524 upper=1.5708 effort=37 velocity=7.33
- joint left_wrist_yaw_joint: limit lower=-1.1344 upper=1.1344 effort=25 velocity=4.44 -> lower=-0.6109 upper=1.1344 effort=20 velocity=6.28; origin xyz=0.021 0 0 rpy=0 0 0 -> xyz=0.23 0 0 rpy=0 0 0; parent left_wrist_pitch_link -> left_wrist_roll_link
- joint right_hand_joint: origin xyz=0.031 0 0 rpy=0 0 0 -> xyz=0.016 0 0 rpy=0 0 0; parent right_wrist_yaw_link -> right_wrist_pitch_link
- joint right_wrist_pitch_joint: limit lower=-0.5236 upper=0.5236 effort=20 velocity=6.28 -> lower=-0.5236 upper=0.5236 effort=25 velocity=4.44; origin xyz=0.23 0 0 rpy=0 0 0 -> xyz=0.021 0 0 rpy=0 0 0; parent right_wrist_roll_link -> right_wrist_yaw_link
- joint right_wrist_roll_joint: limit lower=-2.0071 upper=2.0071 effort=37 velocity=7.33 -> lower=-1.5708 upper=3.7524 effort=37 velocity=7.33
- joint right_wrist_yaw_joint: limit lower=-1.1344 upper=1.1344 effort=25 velocity=4.44 -> lower=-1.1344 upper=0.6109 effort=20 velocity=6.28; origin xyz=0.021 0 0 rpy=0 0 0 -> xyz=0.23 0 0 rpy=0 0 0; parent right_wrist_pitch_link -> right_wrist_roll_link
